File: Ampli_10W_Txutxi_version.sch (KiCad schematic (older format))
At the start: 9 parts, among them U1 TDA2003V

Commit message: Update library and PCB
Parts:
- added 100k1: POT, Potentiometers:Potentiometer_Alps-RK16-single, symbol POT
- C1: footprint (none) -> Capacitors_ThroughHole:C_Radial_D5_L11_P2
- C2: footprint (none) -> Capacitors_ThroughHole:C_Radial_D10_L16_P5
- C3: footprint (none) -> Capacitors_ThroughHole:C_Radial_D13_L21_P5
- CONN_1: renamed from CONN_01; footprint (none) -> Connect:bornier2
- CONN_2: renamed from CONN_02; footprint (none) -> Connect:bornier2
- CONN_3: renamed from CONN_03; footprint (none) -> Connect:bornier2
- R1, R2: footprint (none) -> Resistors_ThroughHole:Resistor_Horizontal_RM10mm
- U1: footprint PW-5 -> TO_SOT_Packages_THT:Pentawatt_Neutral_Staggered_Verical_TO220-5-T05D
Connections:
- wire segments 18 -> 25
Other:
- moved on the sheet: C3, CONN_1, CONN_3
Changed lines of the file:
@@
 LIBS:memory
 LIBS:xilinx
-LIBS:special
 LIBS:microcontrollers
 LIBS:dsp
@@
 LIBS:contrib
 LIBS:valves
-LIBS:TDA2003
-LIBS:TDA2003H
-LIBS:TDA2003V
-LIBS:klavijador-cache
-EELAYER 24 0
+LIBS:Ampli_10W_Txutxi_version-cache
+EELAYER 25 0
 EELAYER END
 $Descr A4 11693 8268
@@
 Sheet 1 1
 Title ""
-Date "3 nov 2013"
+Date "7 jun 2015"
 Rev ""
 Comp ""
@@
 $EndDescr
 $Comp
-L TDA2003V U1
-U 1 1 535AC30F
-P 5450 2450
-F 0 "U1" H 5700 2300 40  0000 C CNN
-F 1 "TDA2003V" H 5700 2250 40  0000 C CNN
-F 2 "PW-5" H 5250 2450 30  0000 C CIN
-F 3 "" H 5450 2450 60  0000 C CNN
-	1    5450 2450
-	1    0    0    -1
-$EndComp
-$Comp
 L CP1 C1
 U 1 1 535AC7D3
@@
 F 0 "C1" H 4050 2600 50  0000 L CNN
 F 1 "10uF" H 4050 2400 50  0000 L CNN
-F 2 "" H 4000 2500 60  0000 C CNN
+F 2 "Capacitors_ThroughHole:C_Radial_D5_L11_P2" H 4000 2500 60  0001 C CNN
 F 3 "" H 4000 2500 60  0000 C CNN
 	1    4000 2500
@@
 	4950 2300 4000 2300
 $Comp
-L GND #PWR6
+L GND #PWR01
 U 1 1 535AC874
 P 5400 3050
-F 0 "#PWR6" H 5400 3050 30  0001 C CNN
+F 0 "#PWR01" H 5400 3050 30  0001 C CNN
 F 1 "GND" H 5400 2980 30  0001 C CNN
 F 2 "" H 5400 3050 60  0000 C CNN
@@
 	5400 2800 5400 3050
 $Comp
-L +9V #PWR5
+L +9V #PWR02
 U 1 1 535AC88B
 P 5400 1950
-F 0 "#PWR5" H 5400 1920 20  0001 C CNN
+F 0 "#PWR02" H 5400 1920 20  0001 C CNN
 F 1 "+9V" H 5400 2060 30  0000 C CNN
 F 2 "" H 5400 1950 60  0000 C CNN
@@
 F 0 "C2" H 4750 2900 50  0000 L CNN
 F 1 "470uF" H 4750 2700 50  0000 L CNN
-F 2 "" H 4700 2800 60  0000 C CNN
+F 2 "Capacitors_ThroughHole:C_Radial_D10_L16_P5" H 4700 2800 60  0001 C CNN
 F 3 "" H 4700 2800 60  0000 C CNN
 F 4 "35V" H 4700 2800 60  0001 C CNN "Tensión"
@@
 F 0 "R1" V 4780 3600 40  0000 C CNN
 F 1 "220" V 4707 3601 40  0000 C CNN
-F 2 "" V 4630 3600 30  0000 C CNN
+F 2 "Resistors_ThroughHole:Resistor_Horizontal_RM10mm" V 4630 3600 30  0001 C CNN
 F 3 "" H 4700 3600 30  0000 C CNN
 	1    4700 3600
@@
 $EndComp
 Wire Wire Line
-	4700 3000 4700 3350
+	4700 2950 4700 3450
 $Comp
 L R R2
@@
 F 0 "R2" V 4180 3600 40  0000 C CNN
 F 1 "2.2" V 4107 3601 40  0000 C CNN
-F 2 "" V 4030 3600 30  0000 C CNN
+F 2 "Resistors_ThroughHole:Resistor_Horizontal_RM10mm" V 4030 3600 30  0001 C CNN
 F 3 "" H 4100 3600 30  0000 C CNN
 	1    4100 3600
@@
 	4700 3200 4100 3200
 Wire Wire Line
-	4100 3200 4100 3350
+	4100 3200 4100 3450
 Connection ~ 4700 3200
 $Comp
-L GND #PWR4
+L GND #PWR03
 U 1 1 535AC9A9
 P 4100 4000
-F 0 "#PWR4" H 4100 4000 30  0001 C CNN
+F 0 "#PWR03" H 4100 4000 30  0001 C CNN
 F 1 "GND" H 4100 3930 30  0001 C CNN
 F 2 "" H 4100 4000 60  0000 C CNN
@@
 $EndComp
 Wire Wire Line
-	4100 3850 4100 4000
-Wire Wire Line
-	5950 2450 6650 2450
-Wire Wire Line
-	6400 2450 6400 3850
-Wire Wire Line
-	6400 3850 4700 3850
+	4100 3750 4100 4000
+Wire Wire Line
+	6200 2450 6200 3850
 $Comp
 L CP1 C3
 U 1 1 535ACA21
-P 6850 2450
-F 0 "C3" H 6900 2550 50  0000 L CNN
-F 1 "1000uF" H 6900 2350 50  0000 L CNN
-F 2 "" H 6850 2450 60  0000 C CNN
-F 3 "" H 6850 2450 60  0000 C CNN
-F 4 "35V" H 6850 2450 60  0001 C CNN "Tensión"
-	1    6850 2450
+P 6500 2450
+F 0 "C3" H 6550 2550 50  0000 L CNN
+F 1 "1000uF" H 6550 2350 50  0000 L CNN
+F 2 "Capacitors_ThroughHole:C_Radial_D13_L21_P5" H 6500 2450 60  0001 C CNN
+F 3 "" H 6500 2450 60  0000 C CNN
+F 4 "35V" H 6500 2450 60  0001 C CNN "Tensión"
+	1    6500 2450
 	0    -1   -1   0
 $EndComp
-Connection ~ 6400 2450
-$Comp
-L CONN_2 CONN_03
+Connection ~ 6200 2450
+$Comp
+L CONN_2 CONN_3
 U 1 1 535ACAC6
-P 7550 2550
-F 0 "CONN_03" V 7500 2550 40  0000 C CNN
-F 1 "Carga 4-8 ohm" V 7600 2550 40  0000 C CNN
-F 2 "" H 7550 2550 60  0000 C CNN
-F 3 "" H 7550 2550 60  0000 C CNN
-	1    7550 2550
-	1    0    0    -1
-$EndComp
-Wire Wire Line
-	7050 2450 7200 2450
-$Comp
-L GND #PWR7
+P 7350 2550
+F 0 "CONN_3" V 7300 2550 40  0000 C CNN
+F 1 "Carga 4-8 ohm" V 7400 2550 40  0000 C CNN
+F 2 "Connect:bornier2" H 7350 2550 60  0001 C CNN
+F 3 "" H 7350 2550 60  0000 C CNN
+	1    7350 2550
+	1    0    0    -1
+$EndComp
+$Comp
+L GND #PWR04
 U 1 1 535ACAE7
-P 7200 2900
-F 0 "#PWR7" H 7200 2900 30  0001 C CNN
-F 1 "GND" H 7200 2830 30  0001 C CNN
-F 2 "" H 7200 2900 60  0000 C CNN
-F 3 "" H 7200 2900 60  0000 C CNN
-	1    7200 2900
-	1    0    0    -1
-$EndComp
-Wire Wire Line
-	7200 2650 7200 2900
-$Comp
-L CONN_2 CONN_01
+P 7000 2900
+F 0 "#PWR04" H 7000 2900 30  0001 C CNN
+F 1 "GND" H 7000 2830 30  0001 C CNN
+F 2 "" H 7000 2900 60  0000 C CNN
+F 3 "" H 7000 2900 60  0000 C CNN
+	1    7000 2900
+	1    0    0    -1
+$EndComp
+Wire Wire Line
+	7000 2650 7000 2900
+$Comp
+L CONN_2 CONN_1
 U 1 1 535ACB15
-P 3050 3000
-F 0 "CONN_01" V 3000 3000 40  0000 C CNN
-F 1 "Audio_In" V 3100 3000 40  0000 C CNN
-F 2 "" H 3050 3000 60  0000 C CNN
-F 3 "" H 3050 3000 60  0000 C CNN
-	1    3050 3000
+P 3050 2750
+F 0 "CONN_1" V 3000 2750 40  0000 C CNN
+F 1 "Audio_In" V 3100 2750 40  0000 C CNN
+F 2 "Connect:bornier2" H 3050 2750 60  0001 C CNN
+F 3 "" H 3050 2750 60  0000 C CNN
+	1    3050 2750
 	-1   0    0    -1
 $EndComp
 Wire Wire Line
-	4000 2700 4000 2900
-Wire Wire Line
-	4000 2900 3400 2900
-$Comp
-L GND #PWR1
+	4000 2650 4000 2900
+$Comp
+L GND #PWR05
 U 1 1 535ACB46
 P 3400 3250
-F 0 "#PWR1" H 3400 3250 30  0001 C CNN
+F 0 "#PWR05" H 3400 3250 30  0001 C CNN
 F 1 "GND" H 3400 3180 30  0001 C CNN
 F 2 "" H 3400 3250 60  0000 C CNN
@@
 $EndComp
 Wire Wire Line
-	3400 3100 3400 3250
-$Comp
-L CONN_2 CONN_02
+	3400 2850 3400 3250
+$Comp
+L CONN_2 CONN_2
 U 1 1 535B38B5
 P 3050 4000
-F 0 "CONN_02" V 3000 4000 40  0000 C CNN
+F 0 "CONN_2" V 3000 4000 40  0000 C CNN
 F 1 "Vcc" V 3100 4000 40  0000 C CNN
-F 2 "" H 3050 4000 60  0000 C CNN
+F 2 "Connect:bornier2" H 3050 4000 60  0001 C CNN
 F 3 "" H 3050 4000 60  0000 C CNN
 	1    3050 4000
@@
 $EndComp
 $Comp
-L +9V #PWR2
+L +9V #PWR06
 U 1 1 535B38CC
 P 3400 3750
-F 0 "#PWR2" H 3400 3720 20  0001 C CNN
+F 0 "#PWR06" H 3400 3720 20  0001 C CNN
 F 1 "+9V" H 3400 3860 30  0000 C CNN
 F 2 "" H 3400 3750 60  0000 C CNN
@@
 	3400 3750 3400 3900
 $Comp
-L GND #PWR3
+L GND #PWR07
 U 1 1 535B38EB
 P 3400 4250
-F 0 "#PWR3" H 3400 4250 30  0001 C CNN
+F 0 "#PWR07" H 3400 4250 30  0001 C CNN
 F 1 "GND" H 3400 4180 30  0001 C CNN
 F 2 "" H 3400 4250 60  0000 C CNN
@@
 Wire Wire Line
 	3400 4100 3400 4250
+$Comp
+L POT 100k1
+U 1 1 55748CCB
+P 3700 2900
+F 0 "100k1" H 3700 2800 50  0000 C CNN
+F 1 "POT" H 3700 2900 50  0000 C CNN
+F 2 "Potentiometers:Potentiometer_Alps-RK16-single" H 3300 3000 60  0000 C CNN
+F 3 "~" H 3700 2900 60  0000 C CNN
+	1    3700 2900
+	0    1    1    0
+$EndComp
+Wire Wire Line
+	4000 2900 3850 2900
+Wire Wire Line
+	3700 3150 3400 3150
+Connection ~ 3400 3150
+Wire Wire Line
+	6650 2450 7000 2450
+Wire Wire Line
+	3400 2650 3700 2650
+Wire Wire Line
+	4700 3850 4700 3750
+Wire Wire Line
+	4000 2300 4000 2350
+Wire Wire Line
+	4700 2600 4700 2650
+$Comp
+L PWR_FLAG #v08
+U 1 1 55785B8F
+P 3550 3750
+F 0 "#v08" H 3550 3845 50  0001 C CNN
+F 1 "PWR_FLAG" H 3550 3930 50  0000 C CNN
+F 2 "" H 3550 3750 60  0000 C CNN
+F 3 "" H 3550 3750 60  0000 C CNN
+	1    3550 3750
+	1    0    0    -1
+$EndComp
+$Comp
+L PWR_FLAG #ground09
+U 1 1 55785BB7
+P 4300 3850
+F 0 "#ground09" H 4300 3945 50  0001 C CNN
+F 1 "PWR_FLAG" H 4300 4030 50  0000 C CNN
+F 2 "" H 4300 3850 60  0000 C CNN
+F 3 "" H 4300 3850 60  0000 C CNN
+	1    4300 3850
+	1    0    0    -1
+$EndComp
+Wire Wire Line
+	4300 3850 4100 3850
+Connection ~ 4100 3850
+Wire Wire Line
+	3550 3750 3400 3750
+Wire Wire Line
+	6200 3850 4700 3850
+Wire Wire Line
+	5950 2450 6350 2450
+$Comp
+L TDA2003V U1
+U 1 1 56D7770D
+P 5450 2450
+F 0 "U1" H 5700 2300 50  0000 C CNN
+F 1 "TDA2003V" H 5700 2250 50  0000 C CNN
+F 2 "TO_SOT_Packages_THT:Pentawatt_Neutral_Staggered_Verical_TO220-5-T05D" H 5250 2450 50  0000 C CIN
+F 3 "" H 5450 2450 50  0000 C CNN
+	1    5450 2450
+	1    0    0    -1
+$EndComp
 $EndSCHEMATC
